Commit message: Add geometry to human urdf for arm and body

File: urdf/human_kinematics.urdf (robot description, URDF)
Before this commit: robot human, 9 links, 8 joints
Links:
- link neck: geometry visual cylinder length=1.47 radius=0.04
- link wrist: geometry visual box size=0.1 0.07 0.017; visual cylinder length=0.51 radius=0.02
